File: PCB_design_try.kicad_sch (KiCad schematic)
At the start: 14 parts

Commit message: Kairo-kannsei
Parts:
- removed R?: 10k, symbol Device:R_Small
- removed SW?: SW_Push, symbol Switch:SW_Push
- added D1, D10, D11, D12, D13, D14, D15, D16, D17, D18, D19, D2, D20, D21, D22, D23, D24, D25, D26, D27, D28, D29, D3, D30, D31, D32, D33, D34, D35, D36, D37, D38, D39, D4, D40, D41, D42, D43, D44, D45, D46, D47, D48, D49, D5, D50, D51, D52, D6, D7, D8, D9: D_Small, Diode_SMD:D_SOD-123, symbol Device:D_Small
- added D53: PRTR5V0U2X, Package_TO_SOT_SMD:SOT-143, symbol Power_Protection:PRTR5V0U2X
- added F1: 500mA, Fuse:Fuse_1206_3216Metric_Pad1.42x1.75mm_HandSolder, symbol Device:Polyfuse_Small
- added J1: USB_C_Receptacle_USB2.0, USB4085-GF-A_REVA-3:GCT_USB4085-GF-A_REVA, symbol Connector:USB_C_Receptacle_USB2.0
- added LS1: Speaker, Buzzer_Beeper:Buzzer_Murata_PKLCS1212E, symbol Device:Speaker
- added R1: 10k, Resistor_SMD:R_0805_2012Metric_Pad1.20x1.40mm_HandSolder, symbol Device:R_Small
- added R3, R4: 5.1k, Resistor_SMD:R_0805_2012Metric_Pad1.20x1.40mm_HandSolder, symbol Device:R_Small
- added R7: 1k, Resistor_SMD:R_0805_2012Metric_Pad1.20x1.40mm_HandSolder, symbol Device:R_Small
- added SW1, SW10, SW11, SW12, SW13, SW14, SW15, SW16, SW17, SW18, SW19, SW2, SW20, SW21, SW22, SW23, SW24, SW25, SW26, SW27, SW28, SW29, SW3, SW30, SW31, SW32, SW33, SW34, SW35, SW36, SW37, SW38, SW39, SW4, SW40, SW41, SW42, SW43, SW44, SW45, SW46, SW47, SW48, SW49, SW5, SW50, SW51, SW52, SW53, SW6, SW7, SW8, SW9: SW_Push, MX_Alps_Hybrid:MX-1U-NoLED, symbol Switch:SW_Push
- added SW54: RotaryEncoder_Switch, Rotary_Encoder:RotaryEncoder_Alps_EC12E-Switch_Vertical_H20mm, symbol Device:RotaryEncoder_Switch
- C1, C2, C3, C4, C5, C6: renamed from C?; footprint (none) -> Capacitor_SMD:C_0805_2012Metric_Pad1.18x1.45mm_HandSolder
- C7: renamed from C?; value 10uF -> 4.7uF; footprint (none) -> Capacitor_SMD:C_0805_2012Metric_Pad1.18x1.45mm_HandSolder
- R2, R5, R6: renamed from R?; footprint (none) -> Resistor_SMD:R_0805_2012Metric_Pad1.20x1.40mm_HandSolder
- Y1: renamed from Y?; footprint (none) -> Crystal:Resonator_SMD_Murata_SFECV-3Pin_6.9x2.9mm
- gave numbers to parts that had none: 1
Connections:
- net +5V: now also F1.2, R1.2
- net D+: now also R5.2
- net D-: now also R6.2
- net GND: now also D53.1 (GND), J1.A1 (GND), J1.A12 (GND), J1.B1 (GND), J1.B12 (GND), J1.S1 (SHIELD), LS1.1, R3.2, R4.2, SW53.1, SW54.C
- net at U1.24 (PC1/~{RESET}): now also R1.1, SW53.2
- net at R6.1: now also D53.3 (I/O2), J1.A7 (D-), J1.B7 (D-)
- net at R5.1: now also D53.2 (I/O1), J1.A6 (D+), J1.B6 (D+)
- net col11: now reaches U1.10 (PD4)
- net col11: now also SW45.1, SW46.1, SW47.1, SW48.1
- net col10: now reaches U1.11 (PD5)
- net col10: now also SW41.1, SW42.1, SW43.1, SW44.1
- net col9: now reaches U1.12 (PD6)
- net col9: now also SW37.1, SW38.1, SW39.1, SW40.1
- net col8: now reaches U1.14 (PB0)
- net col8: now also SW33.1, SW34.1, SW35.1, SW36.1
- net col7: now reaches U1.15 (PB1)
- net col7: now also SW29.1, SW30.1, SW31.1, SW32.1
- net col6: now reaches U1.16 (PB2)
- net col6: now also SW25.1, SW26.1, SW27.1, SW28.1
- net row1: now reaches U1.17 (PB3)
- net row1: now also D10.1 (K), D14.1 (K), D18.1 (K), D2.1 (K), D22.1 (K), D26.1 (K), D30.1 (K), D34.1 (K), D38.1 (K), D42.1 (K), D46.1 (K), D50.1 (K), D6.1 (K)
- net col5: now reaches U1.18 (PB4)
- net col5: now also SW21.1, SW22.1, SW23.1, SW24.1
- net col4: now reaches U1.19 (PB5)
- net col4: now also SW17.1, SW18.1, SW19.1, SW20.1
- net col3: now reaches U1.20 (PB6)
- net col3: now also SW13.1, SW14.1, SW15.1, SW16.1
- net col2: now reaches U1.21 (PB7)
- net col2: now also SW10.1, SW11.1, SW12.1, SW9.1
- net col1: now reaches U1.22 (PC7)
- net col1: now also SW5.1, SW6.1, SW7.1, SW8.1
- net col0: now reaches U1.23 (PC6)
- net col0: now also SW1.1, SW2.1, SW3.1, SW4.1
- net Audio: now reaches U1.25 (PC5)
- net Audio: now also R7.1
- net row0: now reaches U1.26 (PC4)
- net row0: now also D1.1 (K), D13.1 (K), D17.1 (K), D21.1 (K), D25.1 (K), D29.1 (K), D33.1 (K), D37.1 (K), D41.1 (K), D45.1 (K), D49.1 (K), D5.1 (K), D9.1 (K)
- net RE_A: now reaches U1.5 (PC2)
- net RE_A: now also SW54.B
- net RE_B: now reaches U1.6 (PD0)
- net RE_B: now also SW54.A
- net col12: now reaches U1.7 (PD1)
- net col12: now also SW49.1, SW50.1, SW51.1, SW52.1
- net row3: now reaches U1.8 (PD2)
- net row3: now also D12.1 (K), D16.1 (K), D20.1 (K), D24.1 (K), D28.1 (K), D32.1 (K), D36.1 (K), D4.1 (K), D40.1 (K), D44.1 (K), D48.1 (K), D52.1 (K), D8.1 (K)
- net row2: now reaches U1.9 (PD3)
- net row2: now also D11.1 (K), D15.1 (K), D19.1 (K), D23.1 (K), D27.1 (K), D3.1 (K), D31.1 (K), D35.1 (K), D39.1 (K), D43.1 (K), D47.1 (K), D51.1 (K), D7.1 (K)
- new net: D40.2 (A), SW40.2
- new net: D50.2 (A), SW50.2
- new net: D38.2 (A), SW38.2
- new net: D8.2 (A), SW8.2
- new net: D52.2 (A), SW52.2
- new net: J1.B5 (CC2), R3.1
- new net: D33.2 (A), SW33.2
- new net: D18.2 (A), SW18.2
- new net: D41.2 (A), SW41.2
- new net: D12.2 (A), SW12.2
- new net: D19.2 (A), SW19.2
- new net: D48.2 (A), SW48.2
- new net: D17.2 (A), SW17.2
- new net: D16.2 (A), SW16.2
- new net: D1.2 (A), SW1.2
- new net: D14.2 (A), SW14.2
- new net: D46.2 (A), SW46.2
- new net: D31.2 (A), SW31.2
- new net: D26.2 (A), SW26.2
- new net: D9.2 (A), SW9.2
- new net: D6.2 (A), SW6.2
- new net: D7.2 (A), SW7.2
- new net: D47.2 (A), SW47.2
- new net: D25.2 (A), SW25.2
- new net: D30.2 (A), SW30.2
- new net: D5.2 (A), SW5.2
- new net: D20.2 (A), SW20.2
- new net: D37.2 (A), SW37.2
- new net: D27.2 (A), SW27.2
- new net: D23.2 (A), SW23.2
- new net: D42.2 (A), SW42.2
- new net: D15.2 (A), SW15.2
- new net: D45.2 (A), SW45.2
- new net: D32.2 (A), SW32.2
- new net: D4.2 (A), SW4.2
- new net: D10.2 (A), SW10.2
- new net: D34.2 (A), SW34.2
- new net: D36.2 (A), SW36.2
- new net: D24.2 (A), SW24.2
- new net: D51.2 (A), SW51.2
- new net: D3.2 (A), SW3.2
- new net: D49.2 (A), SW49.2
- new net: D2.2 (A), SW2.2
- new net: D11.2 (A), SW11.2
- new net: D39.2 (A), SW39.2
- new net: J1.A5 (CC1), R4.1
- new net: D13.2 (A), SW13.2
- new net: D29.2 (A), SW29.2
- new net: D44.2 (A), SW44.2
- new net: D22.2 (A), SW22.2
- new net: D43.2 (A), SW43.2
- new net: LS1.2, R7.2
- new net: D21.2 (A), SW21.2
- new net: D28.2 (A), SW28.2
- new net: D35.2 (A), SW35.2
- new net RE_1: SW54.S2
- new net RE_2: SW54.S1
- new net VCC: D53.4 (VCC), F1.1, J1.A4 (VBUS), J1.A9 (VBUS), J1.B4 (VBUS), J1.B9 (VBUS)
Other:
- moved on the sheet: C1, C2, C3, C4, C5, C6, C7, R2, R5, R6, U1, Y1

Commit message: 2022/02/03 Update
Parts:
- removed C1, C2: 22pF, Capacitor_SMD:C_0805_2012Metric_Pad1.18x1.45mm_HandSolder, symbol Device:C_Small
- removed C4, C6: 0.1uF, Capacitor_SMD:C_0805_2012Metric_Pad1.18x1.45mm_HandSolder, symbol Device:C_Small
- removed D20, D24, D32: D_Small, Diode_SMD:D_SOD-123, symbol Device:D_Small
- removed SW20, SW24, SW32: SW_Push, MX_Alps_Hybrid:MX-1U-NoLED, symbol Switch:SW_Push
- removed Y1: 16MHz, Crystal:Resonator_SMD_Murata_SFECV-3Pin_6.9x2.9mm, symbol Device:Crystal_GND24_Small
- added Y1: Crystal_GND3_Small, Crystal:Resonator_SMD_Murata_CSTxExxV-3Pin_3.0x1.1mm_HandSoldering, symbol Device:Crystal_GND3_Small
- C1: renamed from C5; footprint Capacitor_SMD:C_0805_2012Metric_Pad1.18x1.45mm_HandSolder -> Capacitor_SMD:C_0603_1608Metric_Pad1.08x0.95mm_HandSolder
- C2: renamed from C3; value 0.1uF -> 10uF; footprint Capacitor_SMD:C_0805_2012Metric_Pad1.18x1.45mm_HandSolder -> Capacitor_SMD:C_0603_1608Metric_Pad1.08x0.95mm_HandSolder
- C3: renamed from C7; value 4.7uF -> 0.1uF; footprint Capacitor_SMD:C_0805_2012Metric_Pad1.18x1.45mm_HandSolder -> Capacitor_SMD:C_0603_1608Metric_Pad1.08x0.95mm_HandSolder
- F1: footprint Fuse:Fuse_1206_3216Metric_Pad1.42x1.75mm_HandSolder -> Fuse:Fuse_0603_1608Metric_Pad1.05x0.95mm_HandSolder
- J1: footprint USB4085-GF-A_REVA-3:GCT_USB4085-GF-A_REVA -> USB-C:USB_C_GCT_USB4085
- LS1: footprint Buzzer_Beeper:Buzzer_Murata_PKLCS1212E -> Buzzer_Beeper:Buzzer_Murata_PKMCS0909E
- R1, R2, R3, R4, R5, R6, R7: footprint Resistor_SMD:R_0805_2012Metric_Pad1.20x1.40mm_HandSolder -> Resistor_SMD:R_0603_1608Metric_Pad0.98x0.95mm_HandSolder
- SW1, SW10, SW11, SW13, SW14, SW15, SW17, SW18, SW19, SW5, SW6, SW7, SW8, SW9: footprint MX_Alps_Hybrid:MX-1U-NoLED -> MX_Only:MXOnly-1U-Hotswap
- SW12, SW2, SW4: footprint MX_Alps_Hybrid:MX-1U-NoLED -> MX_Only:MXOnly-1.25U-Hotswap
- SW16: footprint MX_Alps_Hybrid:MX-1U-NoLED -> MX_Only:MXOnly-2.25U-Hotswap
- SW20: renamed from SW21; footprint MX_Alps_Hybrid:MX-1U-NoLED -> MX_Only:MXOnly-1U-Hotswap
- SW21: renamed from SW22; footprint MX_Alps_Hybrid:MX-1U-NoLED -> MX_Only:MXOnly-1U-Hotswap
- SW22: renamed from SW23; footprint MX_Alps_Hybrid:MX-1U-NoLED -> MX_Only:MXOnly-1U-Hotswap
- SW23: renamed from SW25; footprint MX_Alps_Hybrid:MX-1U-NoLED -> MX_Only:MXOnly-2.75U-Hotswap
- SW24: renamed from SW26; footprint MX_Alps_Hybrid:MX-1U-NoLED -> MX_Only:MXOnly-1U-Hotswap
- SW25: renamed from SW27; footprint MX_Alps_Hybrid:MX-1U-NoLED -> MX_Only:MXOnly-1U-Hotswap
- SW26: renamed from SW28; footprint MX_Alps_Hybrid:MX-1U-NoLED -> MX_Only:MXOnly-1U-Hotswap
- SW27: renamed from SW29; footprint MX_Alps_Hybrid:MX-1U-NoLED -> MX_Only:MXOnly-1U-Hotswap
- SW28: renamed from SW30; footprint MX_Alps_Hybrid:MX-1U-NoLED -> MX_Only:MXOnly-1U-Hotswap
- SW29: renamed from SW31; footprint MX_Alps_Hybrid:MX-1U-NoLED -> MX_Only:MXOnly-1U-Hotswap
- SW3: footprint MX_Alps_Hybrid:MX-1U-NoLED -> MX_Only:MXOnly-1.75U-Hotswap
- SW30: renamed from SW33; footprint MX_Alps_Hybrid:MX-1U-NoLED -> MX_Only:MXOnly-1U-Hotswap
- SW31: renamed from SW34; footprint MX_Alps_Hybrid:MX-1U-NoLED -> MX_Only:MXOnly-1U-Hotswap
- SW32: renamed from SW35; footprint MX_Alps_Hybrid:MX-1U-NoLED -> MX_Only:MXOnly-1U-Hotswap
- SW33: renamed from SW36; footprint MX_Alps_Hybrid:MX-1U-NoLED -> MX_Only:MXOnly-1U-Hotswap
- SW34: renamed from SW37; footprint MX_Alps_Hybrid:MX-1U-NoLED -> MX_Only:MXOnly-1U-Hotswap
- SW35: renamed from SW38; footprint MX_Alps_Hybrid:MX-1U-NoLED -> MX_Only:MXOnly-1U-Hotswap
- SW36: renamed from SW39; footprint MX_Alps_Hybrid:MX-1U-NoLED -> MX_Only:MXOnly-1U-Hotswap
- SW37: renamed from SW40; footprint MX_Alps_Hybrid:MX-1U-NoLED -> MX_Only:MXOnly-1.25U-Hotswap
- SW38: renamed from SW41; footprint MX_Alps_Hybrid:MX-1U-NoLED -> MX_Only:MXOnly-1U-Hotswap
- SW39: renamed from SW42; footprint MX_Alps_Hybrid:MX-1U-NoLED -> MX_Only:MXOnly-1U-Hotswap
- SW40: renamed from SW43; footprint MX_Alps_Hybrid:MX-1U-NoLED -> MX_Only:MXOnly-1U-Hotswap
- SW41: renamed from SW44; footprint MX_Alps_Hybrid:MX-1U-NoLED -> MX_Only:MXOnly-1U-Hotswap
- SW42: renamed from SW45; footprint MX_Alps_Hybrid:MX-1U-NoLED -> MX_Only:MXOnly-1.75U-Hotswap
- SW43: renamed from SW46; footprint MX_Alps_Hybrid:MX-1U-NoLED -> MX_Only:MXOnly-1.5U-Hotswap
- SW44: renamed from SW47; footprint MX_Alps_Hybrid:MX-1U-NoLED -> MX_Only:MXOnly-1U-Hotswap
- SW45: renamed from SW48; footprint MX_Alps_Hybrid:MX-1U-NoLED -> MX_Only:MXOnly-1U-Hotswap
- SW46: renamed from SW49; footprint MX_Alps_Hybrid:MX-1U-NoLED -> MX_Only:MXOnly-1U-Hotswap
- SW47: renamed from SW50; footprint MX_Alps_Hybrid:MX-1U-NoLED -> MX_Only:MXOnly-1U-Hotswap
- SW48: renamed from SW51; footprint MX_Alps_Hybrid:MX-1U-NoLED -> MX_Only:MXOnly-1U-Hotswap
- SW49: renamed from SW52; footprint MX_Alps_Hybrid:MX-1U-NoLED -> MX_Only:MXOnly-1U-Hotswap
- SW50: renamed from SW53; footprint MX_Alps_Hybrid:MX-1U-NoLED -> Button_Switch_SMD:SW_SPST_TL3342
- SW51: renamed from SW54; footprint Rotary_Encoder:RotaryEncoder_Alps_EC12E-Switch_Vertical_H20mm -> kbd_Parts:RotaryEncoder_EC12E
- renumbered D21 to D20, D22 to D21, D23 to D22, D25 to D23, D26 to D24, D27 to D25, D28 to D26, D29 to D27, D30 to D28, D31 to D29, D33 to D30, D34 to D31, D35 to D32, D36 to D33, D37 to D34, D38 to D35, D39 to D36, D40 to D37, D41 to D38, D42 to D39, D43 to D40, D44 to D41, D45 to D42, D46 to D43, D47 to D44, D48 to D45, D49 to D46, D50 to D47, D51 to D48, D52 to D49, D53 to D50
Connections:
- net GND: now also Y1.3
- net RE_1: now also D46.2 (A), SW46.1
- net RE_2: now also SW46.2, SW47.2, SW48.2, SW49.2, U1.7 (PD1)
- net col0: now also SW1.2, SW2.2, SW3.2, SW4.2; no longer SW1.1, SW2.1, SW3.1, SW4.1
- net col1: now also SW5.2, SW6.2, SW7.2, SW8.2; no longer SW5.1, SW6.1, SW7.1, SW8.1
- net col10: now also SW38.2, SW39.2, SW40.2, SW41.2; no longer SW38.1, SW39.1, SW40.1, SW41.1
- net col2: now also SW10.2, SW11.2, SW12.2, SW9.2; no longer SW10.1, SW11.1, SW12.1, SW9.1
- net col3: now also SW13.2, SW14.2, SW15.2, SW16.2; no longer SW13.1, SW14.1, SW15.1, SW16.1
- net col4: now also SW17.2, SW18.2, SW19.2; no longer SW17.1, SW18.1, SW19.1
- net col5: now also SW20.2, SW21.2, SW22.2, SW23.2; no longer SW20.1, SW21.1, SW22.1
- net col6: now also SW24.2, SW25.2, SW26.2; no longer SW23.1, SW24.1, SW25.1, SW26.1
- net col7: now also SW27.2, SW28.2, SW29.2; no longer SW27.1, SW28.1, SW29.1
- net col8: now also SW30.2, SW31.2, SW32.2, SW33.2; no longer SW30.1, SW31.1, SW32.1, SW33.1
- net col9: now also SW34.2, SW35.2, SW36.2, SW37.2; no longer SW34.1, SW35.1, SW36.1, SW37.1
- net row0: now also D24.1 (K); no longer D23.1 (K)
- net row1: now also D25.1 (K); no longer D24.1 (K)
- net row2: now also D26.1 (K); no longer D25.1 (K)
- net row3: now also D23.1 (K); no longer D26.1 (K)
- net at D37.2 (A): now also SW37.1; no longer SW37.2
- net at D47.2 (A): now also SW47.1; no longer SW47.2
- net at D35.2 (A): now also SW35.1; no longer SW35.2
- net at D8.2 (A): now also SW8.1; no longer SW8.2
- net at D49.2 (A): now also SW49.1; no longer SW49.2
- net at D30.2 (A): now also SW30.1; no longer SW30.2
- net at D18.2 (A): now also SW18.1; no longer SW18.2
- net at D38.2 (A): now also SW38.1; no longer SW38.2
- net at D12.2 (A): now also SW12.1; no longer SW12.2
- net at D19.2 (A): now also SW19.1; no longer SW19.2
- net at D17.2 (A): now also SW17.1; no longer SW17.2
- net at D16.2 (A): now also SW16.1; no longer SW16.2
- net at D1.2 (A): now also SW1.1; no longer SW1.2
- net at D14.2 (A): now also SW14.1; no longer SW14.2
- net at D29.2 (A): now also SW29.1; no longer SW29.2
- net at D24.2 (A): now also SW24.1; no longer SW24.2
- net at D9.2 (A): now also SW9.1; no longer SW9.2
- net at D6.2 (A): now also SW6.1; no longer SW6.2
- net at D7.2 (A): now also SW7.1; no longer SW7.2
- net at D23.2 (A): now also SW23.1; no longer SW23.2
- net at D28.2 (A): now also SW28.1; no longer SW28.2
- net at D5.2 (A): now also SW5.1; no longer SW5.2
- net at D34.2 (A): now also SW34.1; no longer SW34.2
- net at D25.2 (A): now also SW25.1; no longer SW25.2
- net at D22.2 (A): now also SW22.1; no longer SW22.2
- net at U1.1 (XTAL1): now also Y1.1
- net at D39.2 (A): now also SW39.1; no longer SW39.2
- net at D15.2 (A): now also SW15.1; no longer SW15.2
- net at D4.2 (A): now also SW4.1; no longer SW4.2
- net at D10.2 (A): now also SW10.1; no longer SW10.2
- net at D31.2 (A): now also SW31.1; no longer SW31.2
- net at D33.2 (A): now also SW33.1; no longer SW33.2
- net at D48.2 (A): now also SW48.1; no longer SW48.2
- net at D3.2 (A): now also SW3.1; no longer SW3.2
- net at D2.2 (A): now also SW2.1; no longer SW2.2
- net at D11.2 (A): now also SW11.1; no longer SW11.2
- net at U1.2 (PC0/XTAL2): now also Y1.2
- net at D36.2 (A): now also SW36.1; no longer SW36.2
- net at D13.2 (A): now also SW13.1; no longer SW13.2
- net at D27.2 (A): now also SW27.1; no longer SW27.2
- net at D41.2 (A): now also SW41.1; no longer SW41.2
- net at D21.2 (A): now also SW21.1; no longer SW21.2
- net at D40.2 (A): now also SW40.1; no longer SW40.2
- net at D20.2 (A): now also SW20.1; no longer SW20.2
- net at D26.2 (A): now also SW26.1; no longer SW26.2
- net at D32.2 (A): now also SW32.1; no longer SW32.2
- removed net col12: SW46.1, SW47.1, SW48.1, SW49.1, U1.7 (PD1)
- no-connect marks 0 -> 2
Other:
- moved on the sheet: C3, D1, D10, D11, D12, D13, D14, D15, D16, D17, D18, D19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
