File: PCB_design_try.kicad_pcb (KiCad board)
At the start: 2 copper layers, 116 parts, among them J1 USB_C_Receptacle_USB2.0, SW1 SW_Push, SW10 SW_Push, SW11 SW_Push, SW12 SW_Push, SW13 SW_Push, SW14 SW_Push, SW15 SW_Push, SW16 SW_Push, SW17 SW_Push, SW18 SW_Push, SW19 SW_Push, SW2 SW_Push, SW20 SW_Push, SW21 SW_Push, SW22 SW_Push, SW23 SW_Push, SW24 SW_Push, SW25 SW_Push, SW26 SW_Push, SW27 SW_Push, SW28 SW_Push, SW29 SW_Push, SW3 SW_Push, SW30 SW_Push, SW31 SW_Push, SW32 SW_Push, SW33 SW_Push, SW34 SW_Push, SW35 SW_Push, SW36 SW_Push, SW37 SW_Push, SW38 SW_Push, SW39 SW_Push, SW4 SW_Push, SW40 SW_Push, SW41 SW_Push, SW42 SW_Push, SW43 SW_Push, SW44 SW_Push, SW45 SW_Push, SW46 SW_Push, SW47 SW_Push, SW48 SW_Push, SW49 SW_Push, SW5 SW_Push, SW50 SW_Push, SW51 RotaryEncoder_Switch, SW6 SW_Push, SW7 SW_Push, SW8 SW_Push, SW9 SW_Push, U1 ATmega32U2-M, Y1 Crystal_GND3_Small

Commit message: pcb finished
Parts:
- removed the SW43 at (250.0, 45.2)
- added J1: Conn_01x03, Connector_Wire:SolderWire-0.1sqmm_1x03_P3.6mm_D0.4mm_OD1mm, F.Cu at (231.0, 30.6)
- added SW45: SW_Push, MX_Only:MXOnly-1U-Hotswap, F.Cu at (254.9, 83.3)
- C1: renamed from C2; value 10uF -> 1uF
- C2: renamed from C1; value 1uF -> 10uF
- D50: footprint Package_TO_SOT_SMD:SOT-143 -> Keebio-Parts:SOT-143B
- J2: renamed from J1; moved to B.Cu
- R2: value 10k -> 1k
- R3: renamed from R7; value 1k -> 10k
- SW12: renamed from SW11; footprint MX_Only:MXOnly-1U-Hotswap -> MX_Only:MXOnly-1.25U-Hotswap
- SW13: renamed from SW12; footprint MX_Only:MXOnly-1.25U-Hotswap -> MX_Only:MXOnly-1U-Hotswap
- SW16: renamed from SW15; footprint MX_Only:MXOnly-1U-Hotswap -> MX_Only:MXOnly-2.25U-Hotswap
- SW17: renamed from SW16; footprint MX_Only:MXOnly-2.25U-Hotswap -> MX_Only:MXOnly-1U-Hotswap
- SW26: footprint MX_Only:MXOnly-1U-Hotswap -> MX_Only:MXOnly-2.75U-Hotswap
- SW27: renamed from SW23; footprint MX_Only:MXOnly-2.75U-Hotswap -> MX_Only:MXOnly-1U-Hotswap
- SW31: renamed from SW51; value RotaryEncoder_Switch -> SW_Push; footprint kbd_Parts:RotaryEncoder_EC12E -> MX_Only:MXOnly-1U-Hotswap
- SW37: renamed from SW35; footprint MX_Only:MXOnly-1U-Hotswap -> MX_Only:MXOnly-1.25U-Hotswap
- SW39: renamed from SW37; footprint MX_Only:MXOnly-1.25U-Hotswap -> MX_Only:MXOnly-1U-Hotswap
- SW42: renamed from SW40; footprint MX_Only:MXOnly-1U-Hotswap -> MX_Only:MXOnly-1.75U-Hotswap
- SW43: renamed from SW41; footprint MX_Only:MXOnly-1U-Hotswap -> MX_Only:MXOnly-1.5U-Hotswap
- SW44: renamed from SW42; footprint MX_Only:MXOnly-1.75U-Hotswap -> MX_Only:MXOnly-1U-Hotswap
- SW5: renamed from SW50; footprint Button_Switch_SMD:SW_SPST_TL3342 -> MX_Only:MXOnly-1U-Hotswap
- SW50: renamed from SW48; footprint MX_Only:MXOnly-1U-Hotswap -> Button_Switch_SMD:SW_SPST_TL3342
- SW51: renamed from SW49; value SW_Push -> RotaryEncoder_Switch; footprint MX_Only:MXOnly-1U-Hotswap -> kbd_Parts:RotaryEncoder_EC12E
- Y1: value Crystal_GND3_Small -> CSTCE16M0V53-R0; footprint Crystal:Resonator_SMD_Murata_CSTxExxV-3Pin_3.0x1.1mm_HandSoldering -> CSTCE16M0V53-R0:OSC_CSTCE16M0V53-R0
- moved SW5 184.2 mm to (50.0, 26.2), turned to 0 degrees
- moved R2 128.3 mm to (136.7, 73.8), turned to 0 degrees
- moved R3 106.6 mm to (230.9, 23.9), turned to 90 degrees
- moved SW31 87.4 mm to (188.3, 45.2), turned to 0 degrees
- moved SW9 58.9 mm to (69.1, 26.2)
- moved SW13 58.4 mm to (88.2, 26.2)
- moved SW27 57.6 mm to (164.4, 26.2)
- moved SW17 57.2 mm to (107.3, 26.2)
- moved SW50 56.7 mm to (234.3, 23.7), turned to -90 degrees
- moved SW51 56.3 mm to (273.4, 27.0), turned to 90 degrees
- moved SW46 42.7 mm to (274.0, 26.2)
- moved SW47 42.7 mm to (274.0, 45.2)
- moved SW35 40.8 mm to (207.3, 45.2)
- moved SW43 40.8 mm to (250.2, 45.2)
- moved SW32 40.7 mm to (197.8, 64.3)
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- renumbered D24 to D23, D25 to D24, D26 to D25, D23 to D26, R3 to R4, R4 to R5, R5 to R6, R6 to R7, SW9 to SW10, SW10 to SW11, SW13 to SW14, SW14 to SW15, SW17 to SW18, SW18 to SW19, SW19 to SW20, SW20 to SW21, SW21 to SW22, SW22 to SW23, SW27 to SW28, SW28 to SW29, SW29 to SW30, SW30 to SW32, SW31 to SW33, SW32 to SW34, SW33 to SW35, SW34 to SW36, SW36 to SW38, SW38 to SW40, SW39 to SW41, SW44 to SW46, SW45 to SW47, SW46 to SW48, SW47 to SW49, SW5 to SW6, SW6 to SW7, SW7 to SW8, SW8 to SW9
Connections:
- C1 pad 1: +5V -> Net-(C1-Pad1)
- C2 pad 1: Net-(C1-Pad1) -> +5V
- D11 pad 2: Net-(SW11-Pad1) -> Net-(D11-Pad2)
- D15 pad 2: Net-(SW15-Pad1) -> Net-(D15-Pad2)
- D16 pad 2: Net-(SW16-Pad1) -> Net-(D16-Pad2)
- D17 pad 2: Net-(SW17-Pad1) -> Net-(D17-Pad2)
- D18 pad 2: Net-(SW18-Pad1) -> Net-(D18-Pad2)
- D20 pad 2: Net-(SW20-Pad1) -> Net-(D20-Pad2)
- D21 pad 2: Net-(SW21-Pad1) -> Net-(D21-Pad2)
- D23 pad 2: Net-(SW24-Pad1) -> Net-(D23-Pad2)
- D24 pad 2: Net-(D25-Pad2) -> Net-(D24-Pad2)
- D25 pad 2: Net-(SW26-Pad1) -> Net-(D25-Pad2)
- D26 pad 2: Net-(D23-Pad2) -> Net-(D26-Pad2)
- D27 pad 2: Net-(SW27-Pad1) -> Net-(D27-Pad2)
- D28 pad 2: Net-(SW28-Pad1) -> Net-(D28-Pad2)
- D29 pad 2: Net-(SW29-Pad1) -> Net-(D29-Pad2)
- D30 pad 2: Net-(SW30-Pad1) -> Net-(D30-Pad2)
- D31 pad 2: Net-(SW31-Pad1) -> Net-(D31-Pad2)
- D32 pad 2: Net-(SW32-Pad1) -> Net-(D32-Pad2)
- D35 pad 2: Net-(SW35-Pad1) -> Net-(D35-Pad2)
- D36 pad 2: Net-(SW36-Pad1) -> Net-(D36-Pad2)
- D37 pad 2: Net-(SW37-Pad1) -> Net-(D37-Pad2)
- D38 pad 2: Net-(SW38-Pad1) -> Net-(D38-Pad2)
- D39 pad 2: Net-(SW39-Pad1) -> Net-(D39-Pad2)
- D40 pad 2: Net-(SW40-Pad1) -> Net-(D40-Pad2)
- D41 pad 2: Net-(SW41-Pad1) -> Net-(D41-Pad2)
- D5 pad 2: Net-(SW5-Pad1) -> Net-(D5-Pad2)
- D50 pad 4: VCC -> +5V
- D7 pad 2: Net-(SW7-Pad1) -> Net-(D7-Pad2)
- D8 pad 2: Net-(SW8-Pad1) -> Net-(D8-Pad2)
- R1 pad 2: +5V -> GND
- R2 pad 1: Net-(R2-Pad1) -> Audio
- R2 pad 2: GND -> Net-(LS1-Pad2)
- R3 pad 1: Audio -> +5V
- R3 pad 2: Net-(LS1-Pad2) -> RESET
- SW10 pad 1: Net-(D9-Pad2) -> Net-(D10-Pad2)
- SW11 pad 1: Net-(D10-Pad2) -> Net-(D11-Pad2)
- SW12 pad 1: Net-(SW11-Pad1) -> Net-(D12-Pad2)
- SW13 pad 1: Net-(D12-Pad2) -> Net-(D13-Pad2)
- SW13 pad 2: col2 -> col3
- SW14 pad 1: Net-(D13-Pad2) -> Net-(D14-Pad2)
- SW15 pad 1: Net-(D14-Pad2) -> Net-(D15-Pad2)
- SW16 pad 1: Net-(SW15-Pad1) -> Net-(D16-Pad2)
- SW17 pad 1: Net-(SW16-Pad1) -> Net-(D17-Pad2)
- SW17 pad 2: col3 -> col4
- SW18 pad 1: Net-(SW17-Pad1) -> Net-(D18-Pad2)
- SW19 pad 1: Net-(SW18-Pad1) -> Net-(D19-Pad2)
- SW20 pad 1: Net-(D19-Pad2) -> Net-(D20-Pad2)
- SW20 pad 2: col4 -> col5
- SW21 pad 1: Net-(SW20-Pad1) -> Net-(D21-Pad2)
- SW22 pad 1: Net-(SW21-Pad1) -> Net-(D22-Pad2)
- SW23 pad 1: Net-(D22-Pad2) -> Net-(D23-Pad2)
- SW23 pad 2: col5 -> col6
- SW24 pad 1: Net-(SW24-Pad1) -> Net-(D24-Pad2)
- SW26 pad 1: Net-(SW26-Pad1) -> Net-(D26-Pad2)
- SW27 pad 1: Net-(D23-Pad2) -> Net-(D27-Pad2)
- SW27 pad 2: col5 -> col7
- SW28 pad 1: Net-(SW27-Pad1) -> Net-(D28-Pad2)
- SW29 pad 1: Net-(SW28-Pad1) -> Net-(D29-Pad2)
- SW30 pad 1: Net-(SW29-Pad1) -> Net-(D30-Pad2)
- SW30 pad 2: col7 -> col8
- SW32 pad 1: Net-(SW30-Pad1) -> Net-(D32-Pad2)
- SW33 pad 1: Net-(SW31-Pad1) -> Net-(D33-Pad2)
- SW34 pad 1: Net-(SW32-Pad1) -> Net-(D34-Pad2)
- SW34 pad 2: col8 -> col9
- SW35 pad 1: Net-(D33-Pad2) -> Net-(D35-Pad2)
- SW35 pad 2: col8 -> col9
- SW36 pad 1: Net-(D34-Pad2) -> Net-(D36-Pad2)
- SW37 pad 1: Net-(SW35-Pad1) -> Net-(D37-Pad2)
- SW38 pad 1: Net-(SW36-Pad1) -> Net-(D38-Pad2)
- SW38 pad 2: col9 -> col10
- SW39 pad 1: Net-(SW37-Pad1) -> Net-(D39-Pad2)
- SW39 pad 2: col9 -> col10
- SW40 pad 1: Net-(SW38-Pad1) -> Net-(D40-Pad2)
- SW41 pad 1: Net-(SW39-Pad1) -> Net-(D41-Pad2)
- SW42 pad 1: Net-(SW40-Pad1) -> col11
- SW42 pad 2: col10 -> Net-(D42-Pad2)
- SW43 pad 1: Net-(SW41-Pad1) -> col11
- SW43 pad 2: col10 -> Net-(D43-Pad2)
- SW44 pad 2: Net-(D42-Pad2) -> Net-(D44-Pad2)
- SW46 pad 1: col11 -> RE_1
- SW46 pad 2: Net-(D44-Pad2) -> RE_2
- SW47 pad 1: col11 -> Net-(D47-Pad2)
- SW47 pad 2: Net-(D45-Pad2) -> RE_2
- SW48 pad 1: RE_1 -> Net-(D48-Pad2)
- SW49 pad 1: Net-(D47-Pad2) -> Net-(D49-Pad2)
- SW5 pad 1: GND -> Net-(D5-Pad2)
- SW5 pad 2: Net-(R1-Pad1) -> col1
- SW50 pad 1: Net-(D48-Pad2) -> GND
- SW50 pad 2: RE_2 -> RESET
- SW6 pad 1: Net-(SW5-Pad1) -> Net-(D6-Pad2)
- SW7 pad 1: Net-(D6-Pad2) -> Net-(D7-Pad2)
- SW8 pad 1: Net-(SW7-Pad1) -> Net-(D8-Pad2)
- SW9 pad 1: Net-(SW8-Pad1) -> Net-(D9-Pad2)
- SW9 pad 2: col1 -> col2
- U1 pad 13: Net-(R2-Pad1) -> Net-(R1-Pad1)
- U1 pad 24: Net-(R1-Pad1) -> RESET
- Y1 pad 2: Net-(U1-Pad2) -> GND
- Y1 pad 3: GND -> Net-(U1-Pad2)
Routing:
- net row1: track 0.00 -> 274.7 mm, vias 0 -> 13
- net row0: track 0.00 -> 267.0 mm, vias 0 -> 13
- net col2: track 0.00 -> 266.2 mm, vias 0 -> 2
- net col3: track 0.00 -> 247.1 mm, vias 0 -> 2
- net col0: track 65.4 -> 295.5 mm, vias 0 -> 2
- net col1: track 76.5 -> 285.0 mm, vias 0 -> 2
- net GND: track 147.8 -> 336.0 mm, vias 3 -> 9
- net col4: track 51.2 -> 199.3 mm, vias 0 -> 2
- net col5: track 51.0 -> 178.9 mm, vias 0 -> 2
- net col6: track 75.9 -> 190.5 mm, vias 0 -> 2
- net col7: track 50.8 -> 147.5 mm, vias 0 -> 2
- net +5V: track 17.8 -> 104.2 mm, vias 1 -> 3
- net col8: track 73.9 -> 153.0 mm, vias 0 -> 2
- net RESET: track 0.00 -> 62.7 mm, vias 0 -> 3
- net col9: track 74.6 -> 133.3 mm, vias 0 -> 2
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- added copper zone on B.Cu, net GND
Other:
- board outline added: 261.9 x 77.3 mm
